Commit message: Use meshes in collision_svg instead of the ones in collision

File: urdf/ur5_robot.urdf (robot description, URDF)
Before this commit: robot ur5, 8 links, 7 joints
Links:
- link base_link: geometry collision mesh filename=package://ur_description/meshes/ur5/collision_svg/Base.dae; visual mesh filename=package://ur_description/meshes/ur5/visual/Base.dae
- link forearm_link: geometry collision mesh filename=package://ur_description/meshes/ur5/collision_svg/Forearm.d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; visual mesh filename=package://ur_description/meshes/ur5/visual/Forearm.dae
- link shoulder_link: geometry collision mesh filename=package://ur_description/meshes/ur5/collision_svg/Shoulder.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; visual mesh filename=package://ur_description/meshes/ur5/visual/Shoulder.dae
- link upper_arm_link: geometry collision mesh filename=package://ur_description/meshes/ur5/collision_svg/UpperArm.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; visual mesh filename=package://ur_description/meshes/ur5/visual/UpperArm.dae
- link wrist_1_link: geometry collision mesh filename=package://ur_description/meshes/ur5/collision_svg/Wrist1.dae; visual mesh filename=package://ur_description/meshes/ur5/visual/Wrist1.dae
- link wrist_2_link: geometry collision mesh filename=package://ur_description/meshes/ur5/collision_svg/Wrist2.dae; visual mesh filename=package://ur_description/meshes/ur5/visual/Wrist2.dae
- link wrist_3_link: geometry collision mesh filename=package://ur_description/meshes/ur5/collision_svg/Wrist3.dae; visual mesh filename=package://ur_description/meshes/ur5/visual/Wrist3.dae
