Commit message: Use collision_svg meshes in ur5.urdf.xacro

File: urdf/ur5.urdf.xacro (robot description, xacro)
@@ -77,5 +77,5 @@
       <collision>
         <geometry>
-          <mesh filename="package://ur_description/meshes/ur5/collision/Base.dae" />
+          <mesh filename="package://ur_description/meshes/ur5/collision_svg/Base.dae" />
         </geometry>
       </collision>
@@ -105,5 +105,5 @@
       <collision>
         <geometry>
-          <mesh filename="package://ur_description/meshes/ur5/collision/Shoulder.dae" />
+          <mesh filename="package://ur_description/meshes/ur5/collision_svg/Shoulder.dae" />
         </geometry>
       </collision>
@@ -133,5 +133,5 @@
       <collision>
         <geometry>
-          <mesh filename="package://ur_description/meshes/ur5/collision/UpperArm.dae" />
+          <mesh filename="package://ur_description/meshes/ur5/collision_svg/UpperArm.dae" />
         </geometry>
       </collision>
@@ -161,5 +161,5 @@
       <collision>
         <geometry>
-          <mesh filename="package://ur_description/meshes/ur5/collision/Forearm.dae" />
+          <mesh filename="package://ur_description/meshes/ur5/collision_svg/Forearm.dae" />
         </geometry>
       </collision>
@@ -189,5 +189,5 @@
       <collision>
         <geometry>
-          <mesh filename="package://ur_description/meshes/ur5/collision/Wrist1.dae" />
+          <mesh filename="package://ur_description/meshes/ur5/collision_svg/Wrist1.dae" />
         </geometry>
       </collision>
@@ -217,5 +217,5 @@
       <collision>
         <geometry>
-          <mesh filename="package://ur_description/meshes/ur5/collision/Wrist2.dae" />
+          <mesh filename="package://ur_description/meshes/ur5/collision_svg/Wrist2.dae" />
         </geometry>
       </collision>
@@ -245,5 +245,5 @@
       <collision>
         <geometry>
-          <mesh filename="package://ur_description/meshes/ur5/collision/Wrist3.dae" />
+          <mesh filename="package://ur_description/meshes/ur5/collision_svg/Wrist3.dae" />
         </geometry>
       </collision>
